Commit message: intial commit

File: urdf/agrorob_urdf.urdf (robot description, URDF)
Before this commit: robot agrorob-simplified-assem, 9 links, 8 joints
Links:
- link Wheel_FL: geometry collision mesh filename=package://agrorob_urdf/meshes/Wheel_FL.STL; visual mesh filename=package://agrorob_urdf/meshes/Wheel_FL.STL
- link body: geometry collision mesh filename=package://agrorob_urdf/meshes/body.STL; visual mesh filename=package://agrorob_urdf/meshes/body.STL
- link shin_FL: geometry collision mesh filename=package://agrorob_urdf/meshes/shin_FL.STL; visual mesh filename=package://agrorob_urdf/meshes/shin_FL.STL
- link shin_FR: geometry collision mesh filename=package://agrorob_urdf/meshes/shin_FR.STL; visual mesh filename=package://agrorob_urdf/meshes/shin_FR.STL
- link shin_RL: geometry collision mesh filename=package://agrorob_urdf/meshes/shin_RL.STL; visual mesh filename=package://agrorob_urdf/meshes/shin_RL.STL
- link shin_RR: geometry collision mesh filename=package://agrorob_urdf/meshes/shin_RR.STL; visual mesh filename=package://agrorob_urdf/meshes/shin_RR.STL
- link wheel_FR: geometry collision mesh filename=package://agrorob_urdf/meshes/wheel_FR.STL; visual mesh filename=package://agrorob_urdf/meshes/wheel_FR.STL
- link wheel_RL: geometry collision mesh filename=package://agrorob_urdf/meshes/wheel_RL.STL; visual mesh filename=package://agrorob_urdf/meshes/wheel_RL.STL
- link wheel_RR: geometry collision mesh filename=package://agrorob_urdf/meshes/wheel_RR.STL; visual mesh filename=package://agrorob_urdf/meshes/wheel_RR.STL

Commit message: partially ok, main body has wrong inertia

File: urdf/agrorob_urdf.urdf (robot description, URDF)
Before this commit: robot agrorob_urdf, 9 links, 8 joints
Links:
- link body: geometry collision mesh filename=package://agrorob_urdf/meshes/body.STL; visual mesh filename=file://agrorob_urdf/meshes/body.STL

Commit message: urdf corrected

File: urdf/agrorob_urdf.urdf (robot description, URDF)
Before this commit: robot agrorob_urdf, 9 links, 8 joints
Links:
- removed link Wheel_FL
- removed link body
- added link base_link, mass 109.44; collision mesh filename=package://agrorob_urdf/meshes/base_link.STL; visual mesh filename=package://agrorob_urdf/meshes/base_link.STL
- added link wheel_FL, mass 15.288; collision mesh filename=package://agrorob_urdf/meshes/wheel_FL.STL; visual mesh filename=package://agrorob_urdf/meshes/wheel_FL.STL
- link shin_RL: mass 0 -> 13.879
- link wheel_RR: mass 15.288 -> 15.2882363411273
Joints:
- joint body_shin_FL: origin xyz=1.5 0.9 -0.29141 rpy=0 0 -0.16579 -> xyz=1.4791 0.88866 -0.59348 rpy=0 0 0; parent body -> base_link
- joint body_shin_FR: origin xyz=1.5 -0.9 -0.29141 rpy=0 0 0.1123 -> xyz=1.4791 -0.91134 -0.59348 rpy=0 0 0; parent body -> base_link
- joint body_shin_RL: origin xyz=-1.5 0.9 -0.29141 rpy=0 0 0.10135 -> xyz=-1.5189 0.88866 -0.59348 rpy=0 0 0; parent body -> base_link
- joint body_shin_RR: origin xyz=-1.5 -0.9 -0.29141 rpy=0 0 0.057689 -> xyz=-1.5189 -0.91134 -0.59348 rpy=0 0 0; parent body -> base_link
- joint shin_wheel_FL: child Wheel_FL -> wheel_FL; origin xyz=0 0 -0.62885 rpy=0 -0.94396 0 -> xyz=0 0 -0.62885 rpy=0 0 0
- joint shin_wheel_FR: origin xyz=0 0 -0.62885 rpy=0 0.34975 0 -> xyz=0 0 -0.62885 rpy=0 0 0
- joint shin_wheel_RL: origin xyz=0 0 -0.62885 rpy=-3.1416 0.63844 -3.1416 -> xyz=0 0 -0.62885 rpy=0 0 0
- joint shin_wheel_RR: origin xyz=0 0 -0.62885 rpy=3.1416 0.71165 3.1416 -> xyz=0 0 -0.62885 rpy=0 0 0
