Commit message: major implementation, rviz robot ok

File: urdf/agrorob_visualization.urdf (robot description, URDF)
Before this commit: robot agrorob_urdf, 9 links, 8 joints
Links:
- link base_link: geometry collision mesh filename=package://agrorob_visualization/meshes/base_link.STL; visual mesh filename=package://agrorob_visualization/meshes/base_link.STL
- link shin_FL: geometry collision mesh filename=package://agrorob_visualization/meshes/shin_FL.STL; visual mesh filename=package://agrorob_visualization/meshes/shin_FL.STL
- link shin_FR: geometry collision mesh filename=package://agrorob_visualization/meshes/shin_FR.STL; visual mesh filename=package://agrorob_visualization/meshes/shin_FR.STL
- link shin_RL: geometry collision mesh filename=package://agrorob_visualization/meshes/shin_RL.STL; visual mesh filename=package://agrorob_visualization/meshes/shin_RL.STL
- link shin_RR: geometry collision mesh filename=package://agrorob_visualization/meshes/shin_RR.STL; visual mesh filename=package://agrorob_visualization/meshes/shin_RR.STL
- link wheel_FL: geometry collision mesh filename=package://agrorob_visualization/meshes/wheel_FL.STL; visual mesh filename=package://agrorob_visualization/meshes/wheel_FL.STL
- link wheel_FR: geometry collision mesh filename=package://agrorob_visualization/meshes/wheel_FR.STL; visual mesh filename=package://agrorob_visualization/meshes/wheel_FR.STL
- link wheel_RL: geometry collision mesh filename=package://agrorob_visualization/meshes/wheel_RL.STL; visual mesh filename=package://agrorob_visualization/meshes/wheel_RL.STL
- link wheel_RR: geometry collision mesh filename=package://agrorob_visualization/meshes/wheel_RR.STL; visual mesh filename=package://agrorob_visualization/meshes/wheel_RR.STL
